File: Electronics/03_MotorStage_v1/03_MotorStage_v1.brd (EAGLE design)
At the start: 100 x 80 mm, 73 parts, among them J1 BARRIER_BLOCK-2PIN, J2 BARRIER_BLOCK-5PIN, J3 CONN_2X3_SMD, U1 XL4016-DEV

Commit message: Motor stage circuit board v1 final
Parts:
- moved C9 0.92 mm to (101.5, 66.0)
- turned R34 to 270 degrees
Routing:
- net GND: track 57.7 -> 271.0 mm, vias 0 -> 11
- net V+: track 213.8 -> 210.6 mm
- net N$20: track 10.4 -> 13.1 mm
- net OUT1: track 130.7 -> 128.9 mm
- net N$19: track 3.56 -> 5.13 mm
- net N$15: track 24.7 -> 24.0 mm
- net N$5: track 33.9 -> 34.5 mm
- net OUT4: track 208.0 -> 208.5 mm
Other:
- board text added: "+"
- board text added: "GND-"
- board text added: "IN+"
- board text added: "V+"
- board text added: "ek robotgrrl Jul 9, '22"
- board text added: "gnd"
- board text added: "hippo-ps motor v1"
- board text added: "out1"
- board text added: "out2"
- board text added: "out3"
- board text added: "out4"
- board text added: "swtch"

Commit message: Naming update to Hippo-PD
Other:
- board text added: "hippo-pd motor v1"
- board text removed: "hippo-ps motor v1"
Changed lines of the file:
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@@
 <text x="51.562" y="93.472" size="1.524" layer="22" font="vector" ratio="20" rot="MR180">gnd</text>
 <text x="43.434" y="93.345" size="1.524" layer="22" font="vector" ratio="20" rot="MR180">V+</text>
-<text x="28.702" y="35.052" size="1.524" layer="22" font="vector" ratio="20" rot="MR90">hippo-ps motor v1</text>
+<text x="28.702" y="35.052" size="1.524" layer="22" font="vector" ratio="20" rot="MR90">hippo-pd motor v1</text>
 <text x="28.702" y="62.103" size="1.524" layer="22" font="vector" ratio="20" rot="MR90">ek robotgrrl Jul 9, '22</text>
 </plain>
