File: Electronics/03_MotorStage_v1/03_MotorStage_v1.brd (EAGLE design)
At the start: 100 x 80 mm, 73 parts, among them J1 BARRIER_BLOCK-2PIN, J2 BARRIER_BLOCK-5PIN, J3 CONN_2X3_SMD, U1 XL4016-DEV

Commit message: Updated refdes of some components
Parts:
- renumbered R1 to U2, R14 to U3, R23 to U4, R32 to U5, U$1 to C12, U$2 to C11, U$3 to C13, U$4 to C14
Changed lines of the file:
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@@
 <?xml version="1.0" encoding="utf-8"?>
 <!DOCTYPE eagle SYSTEM "eagle.dtd">
-<eagle version="9.6.2">
+<eagle version="9.5.2">
 <drawing>
 <settings>
-<setting alwaysvectorfont="yes"/>
+<setting alwaysvectorfont="no"/>
 <setting verticaltext="up"/>
 </settings>
@@
 <attribute name="VALUE" x="160.655" y="44.577" size="1.778" layer="26" font="vector" ratio="14" rot="MR270"/>
 </element>
-<element name="U$2" library="Hippo-PS" package="ELECTROLYTIC_CAP" value="100 uF" x="33.782" y="80.772" smashed="yes" rot="MR180">
+<element name="C11" library="Hippo-PS" package="ELECTROLYTIC_CAP" value="100 uF" x="33.782" y="80.772" smashed="yes" rot="MR180">
 <attribute name="AVAILABILITY" value="In Stock" x="33.782" y="80.772" size="1.778" layer="28" rot="MR180" display="off"/>
 <attribute name="DESCRIPTION" value=" 100 µF 35 V Aluminum Electrolytic Capacitors Radial, Can - SMD - 2000 Hrs @ 105°C " x="33.782" y="80.772" size="1.778" layer="28" rot="MR180" display="off"/>
@@
 <attribute name="VALUE" x="158.546" y="72.328" size="1.27" layer="27" font="vector" ratio="14"/>
 </element>
-<element name="R1" library="Hippo-PS" package="AZ1084C" value="AZ1084C" x="48.514" y="79.756" smashed="yes" rot="MR0">
+<element name="U2" library="Hippo-PS" package="AZ1084C" value="AZ1084C" x="48.514" y="79.756" smashed="yes" rot="MR0">
 <attribute name="NAME" x="52.019540625" y="86.015890625" size="1.778" layer="26" font="vector" ratio="14" rot="MR0"/>
 <attribute name="VALUE" x="169.239390625" y="56.00306875" size="1.778" layer="28" font="vector" ratio="14" rot="MR0"/>
@@
 <attribute name="VALUE" x="40.513" y="25.019" size="0.4064" layer="28" font="vector" rot="MR180"/>
 </element>
-<element name="U$1" library="Hippo-PS" package="ELECTROLYTIC_CAP" value="100 uF" x="78.994" y="76.2" smashed="yes" rot="MR270">
+<element name="C12" library="Hippo-PS" package="ELECTROLYTIC_CAP" value="100 uF" x="78.994" y="76.2" smashed="yes" rot="MR270">
 <attribute name="AVAILABILITY" value="In Stock" x="78.994" y="88.138" size="1.778" layer="28" rot="MR270" display="off"/>
 <attribute name="DESCRIPTION" value=" 100 µF 35 V Aluminum Electrolytic Capacitors Radial, Can - SMD - 2000 Hrs @ 105°C " x="78.994" y="88.138" size="1.778" layer="28" rot="MR270" display="off"/>
@@
 <attribute name="PURCHASE-URL" value="https://pricing.snapeda.com/search/part/865080545012/?ref=eda" x="78.994" y="88.138" size="1.778" layer="28" rot="MR270" display="off"/>
 </element>
-<element name="R14" library="Hippo-PS" package="AZ1084C" value="AZ1084C" x="64.77" y="83.82" smashed="yes" rot="MR180">
+<element name="U3" library="Hippo-PS" package="AZ1084C" value="AZ1084C" x="64.77" y="83.82" smashed="yes" rot="MR180">
 <attribute name="NAME" x="61.264459375" y="77.560109375" size="1.778" layer="26" font="vector" ratio="14" rot="MR180"/>
 <attribute name="VALUE" x="158.801609375" y="67.82193125" size="1.778" layer="28" font="vector" ratio="14" rot="MR180"/>
@@
 <attribute name="VALUE" x="46.863" y="25.019" size="0.4064" layer="28" font="vector" rot="MR180"/>
 </element>
-<element name="U$3" library="Hippo-PS" package="ELECTROLYTIC_CAP" value="100 uF" x="103.378" y="86.106" smashed="yes" rot="MR90">
+<element name="C13" library="Hippo-PS" package="ELECTROLYTIC_CAP" value="100 uF" x="103.378" y="86.106" smashed="yes" rot="MR90">
 <attribute name="AVAILABILITY" value="In Stock" x="103.378" y="74.168" size="1.778" layer="28" rot="MR90" display="off"/>
 <attribute name="DESCRIPTION" value=" 100 µF 35 V Aluminum Electrolytic Capacitors Radial, Can - SMD - 2000 Hrs @ 105°C " x="103.378" y="74.168" size="1.778" layer="28" rot="MR90" display="off"/>
@@
 <attribute name="PURCHASE-URL" value="https://pricing.snapeda.com/search/part/865080545012/?ref=eda" x="103.378" y="74.168" size="1.778" layer="28" rot="MR90" display="off"/>
 </element>
-<element name="R23" library="Hippo-PS" package="AZ1084C" value="AZ1084C" x="86.614" y="80.772" smashed="yes" rot="MR0">
+<element name="U4" library="Hippo-PS" package="AZ1084C" value="AZ1084C" x="86.614" y="80.772" smashed="yes" rot="MR0">
 <attribute name="NAME" x="90.119540625" y="87.031890625" size="1.778" layer="26" font="vector" ratio="14" rot="MR0"/>
 <attribute name="VALUE" x="168.985390625" y="63.11506875" size="1.778" layer="28" font="vector" ratio="14" rot="MR0"/>
@@
 <attribute name="VALUE" x="53.213" y="24.765" size="0.4064" layer="28" font="vector" rot="MR180"/>
 </element>
-<element name="U$4" library="Hippo-PS" package="ELECTROLYTIC_CAP" value="100 uF" x="112.776" y="82.042" smashed="yes" rot="MR270">
+<element name="C14" library="Hippo-PS" package="ELECTROLYTIC_CAP" value="100 uF" x="112.776" y="82.042" smashed="yes" rot="MR270">
 <attribute name="AVAILABILITY" value="In Stock" x="112.776" y="93.98" size="1.778" layer="28" rot="MR270" display="off"/>
 <attribute name="DESCRIPTION" value=" 100 µF 35 V Aluminum Electrolytic Capacitors Radial, Can - SMD - 2000 Hrs @ 105°C " x="112.776" y="93.98" size="1.778" layer="28" rot="MR270" display="off"/>
@@
 <attribute name="PURCHASE-URL" value="https://pricing.snapeda.com/search/part/865080545012/?ref=eda" x="112.776" y="93.98" size="1.778" layer="28" rot="MR270" display="off"/>
 </element>
-<element name="R32" library="Hippo-PS" package="AZ1084C" value="AZ1084C" x="105.918" y="68.834" smashed="yes" rot="MR0">
+<element name="U5" library="Hippo-PS" package="AZ1084C" value="AZ1084C" x="105.918" y="68.834" smashed="yes" rot="MR0">
 <attribute name="NAME" x="109.423540625" y="75.093890625" size="1.778" layer="26" font="vector" ratio="14" rot="MR0"/>
 <attribute name="VALUE" x="169.112390625" y="59.68606875" size="1.778" layer="28" font="vector" ratio="14" rot="MR0"/>
@@
 <signal name="V+">
 <contactref element="J1" pad="P$1"/>
-<contactref element="R1" pad="3"/>
+<contactref element="U2" pad="3"/>
 <contactref element="C3" pad="2"/>
 <wire x1="46.228" y1="75.496" x2="43.564" y2="78.16" width="1.524" layer="16"/>
 <wire x1="43.18" y1="78.16" x2="43.564" y2="78.16" width="1.27" layer="16"/>
-<contactref element="R14" pad="3"/>
+<contactref element="U3" pad="3"/>
 <contactref element="C5" pad="2"/>
 <wire x1="70.104" y1="90.242" x2="69.218" y2="90.242" width="1.27" layer="16"/>
 <wire x1="69.218" y1="90.242" x2="67.056" y2="88.08" width="1.524" layer="16"/>
-<contactref element="R23" pad="3"/>
+<contactref element="U4" pad="3"/>
 <contactref element="C7" pad="2"/>
 <wire x1="84.03153125" y1="76.21553125" x2="84.002" y2="76.1003" width="1.27" layer="16"/>
 <wire x1="84.002" y1="76.1003" x2="84.002" y2="72.644" width="1.524" layer="16"/>
 <wire x1="84.328" y1="76.512" x2="84.03153125" y2="76.21553125" width="1.27" layer="16"/>
-<contactref element="R32" pad="3"/>
+<contactref element="U5" pad="3"/>
 <contactref element="C9" pad="2"/>
 <wire x1="101.473" y1="64.19" x2="101.597" y2="64.066" width="1.27" layer="16"/>
@@
 </signal>
 <signal name="OUT1">
-<contactref element="U$2" pad="+"/>
-<contactref element="R1" pad="2"/>
+<contactref element="C11" pad="+"/>
+<contactref element="U2" pad="2"/>
 <contactref element="C4" pad="2"/>
 <contactref element="R2" pad="1"/>
@@
 <signal name="GND">
 <contactref element="J1" pad="P$2"/>
-<contactref element="U$2" pad="-"/>
+<contactref element="C11" pad="-"/>
 <contactref element="C4" pad="1"/>
 <contactref element="D1" pad="P$2"/>
@@
 <contactref element="R5" pad="2"/>
 <contactref element="R8" pad="1"/>
-<contactref element="U$1" pad="-"/>
+<contactref element="C12" pad="-"/>
 <contactref element="C6" pad="1"/>
 <contactref element="D2" pad="P$2"/>
@@
 <contactref element="R18" pad="2"/>
 <contactref element="R21" pad="1"/>
-<contactref element="U$3" pad="-"/>
+<contactref element="C13" pad="-"/>
 <contactref element="C8" pad="1"/>
 <contactref element="D3" pad="P$2"/>
@@
 <contactref element="R27" pad="2"/>
 <contactref element="R30" pad="1"/>
-<contactref element="U$4" pad="-"/>
+<contactref element="C14" pad="-"/>
 <contactref element="C10" pad="1"/>
 <contactref element="D4" pad="P$2"/>
@@
 <signal name="N$5">
 <contactref element="R3" pad="2"/>
-<contactref element="R1" pad="1"/>
+<contactref element="U2" pad="1"/>
 <contactref element="R4" pad="1"/>
 <wire x1="55.753" y1="72.023" x2="50.8" y2="72.023" width="1.524" layer="16"/>
@@
 </signal>
 <signal name="OUT2">
-<contactref element="U$1" pad="+"/>
-<contactref element="R14" pad="2"/>
+<contactref element="C12" pad="+"/>
+<contactref element="U3" pad="2"/>
 <contactref element="C6" pad="2"/>
 <contactref element="R15" pad="1"/>
@@
 <signal name="N$12">
 <contactref element="R16" pad="2"/>
-<contactref element="R14" pad="1"/>
+<contactref element="U3" pad="1"/>
 <contactref element="R17" pad="1"/>
 <wire x1="62.484" y1="88.08" x2="61.214" y2="88.08" width="1.524" layer="16"/>
@@
 <signal name="N$15">
 <contactref element="R25" pad="2"/>
-<contactref element="R23" pad="1"/>
+<contactref element="U4" pad="1"/>
 <contactref element="R26" pad="1"/>
 <wire x1="94.488" y1="87.194" x2="96.41" y2="85.272" width="1.524" layer="16"/>
@@
 </signal>
 <signal name="OUT3">
-<contactref element="U$3" pad="+"/>
-<contactref element="R23" pad="2"/>
+<contactref element="C13" pad="+"/>
+<contactref element="U4" pad="2"/>
 <contactref element="C8" pad="2"/>
 <contactref element="R24" pad="1"/>
@@
 <signal name="N$20">
 <contactref element="R34" pad="2"/>
-<contactref element="R32" pad="1"/>
+<contactref element="U5" pad="1"/>
 <contactref element="R35" pad="1"/>
 <wire x1="114.808" y1="69.414" x2="114.808" y2="67.564" width="1.524" layer="16"/>
@@
 </signal>
 <signal name="OUT4">
-<contactref element="U$4" pad="+"/>
-<contactref element="R32" pad="2"/>
+<contactref element="C14" pad="+"/>
+<contactref element="U5" pad="2"/>
 <contactref element="C10" pad="2"/>
 <contactref element="R33" pad="1"/>
