File: Electronics/05_ServoStage_v1/05_ServoStage_v1.sch (EAGLE design)
At the start: 58 parts, among them J1 SCREW_TERMINAL_4, J2 BARRIER_BLOCK-4PIN, J3 CONN_2X3_SMD, U1 XL4005-DEV, U2 XL4005-DEV

Commit message: Servo stage: Completed routing
Parts:
- removed TP6, TP9: TP, Hippo-PS:TP
Connections:
- net N$17: now also J1.P$4, J2.P$3, TP8.P$1; no longer J1.P$3, J2.P$4
- net N$18: now also J1.P$3, J2.P$4, TP7.P$1; no longer J1.P$4, J2.P$3
- net N$2: now also TP5.P$1
- net NEOPIXELS: no longer TP5.P$1
- net OUT1: no longer TP6.P$1, TP7.P$1
- net OUT2: no longer TP8.P$1, TP9.P$1
- net SIG1: now also J3.P$3; no longer J3.P$1
- net SIG2: now also J3.P$5; no longer J3.P$2
- net SIG_SMPS: now also J3.P$1; no longer J3.P$3
Other:
- note added: "LEDs"
- note added: "Voltage Dividers for SMPS"
- note removed: "Voltage Divider and LED (for switching regulator)"
- moved on the sheet: F1, F2, F3, H1, H2, H3, H4, J1, J2, J3, TP1, TP2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

Commit message: Naming update to Hippo-PD
Other:
- note added: "Hippo-PD Servo Stage Designed by: Erin Kennedy July 14, 2022"
- note removed: "Hippo-PS Servo Stage Designed by: Erin Kennedy July 14, 2022"
Changed lines of the file:
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@@
 <text x="172.72" y="114.3" size="2.54" layer="95">Output of Regulators</text>
 <text x="53.34" y="35.56" size="2.54" layer="95">Brass Standoffs</text>
-<text x="149.86" y="25.4" size="1.778" layer="95">Hippo-PS Servo Stage
+<text x="149.86" y="25.4" size="1.778" layer="95">Hippo-PD Servo Stage
 Designed by: Erin Kennedy
 July 14, 2022</text>
@@
 <plain>
 <text x="55.88" y="170.18" size="2.54" layer="95">Linear Regulator (5.2V)</text>
-<text x="149.86" y="25.4" size="1.778" layer="95">Hippo-PS Servo Stage
+<text x="149.86" y="25.4" size="1.778" layer="95">Hippo-PD Servo Stage
 Designed by: Erin Kennedy
 July 14, 2022</text>
