File: Electronics/00_CoverStage_v1/00_CoverStage_v1.sch (EAGLE design)
At the start: 0 parts

Commit message: Cover stage artwork naming update
Other:
- note added: "Hippo-PD Cover Stage Designed by: Erin Kennedy July 12, 2022"
- note removed: "Hippo-PS Cover Stage Designed by: Erin Kennedy July 12, 2022"
Changed lines of the file:
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@@
 <sheet>
 <plain>
-<text x="151.638" y="25.654" size="1.778" layer="95">Hippo-PS Cover Stage
+<text x="151.638" y="25.654" size="1.778" layer="95">Hippo-PD Cover Stage
 Designed by: Erin Kennedy
 July 12, 2022 </text>
