File: Electronics/02_MonitorStage_v1/02_MonitorStage_v1.brd (EAGLE design)
At the start: 100 x 80 mm, 58 parts, among them J1 CONN_2X3_SMD, J2 BARRIER_BLOCK-2PIN, J3 CONN_2X3_SMD, J4 CONN_2X3_SMD, J5 CONN_2X3_SMD, J6 CONN_2X3_SMD, J7 CONN_2X3_SMD, Q1 PN2222A-SOT-23

Commit message: Monitor stage electronics v1 final
Other:
- board text added: "GND"
- board text added: "IN+"
- board text added: "ek robotgrrl Jul 22, '22"
- board text added: "hippo-pd monitor v1"
Changed lines of the file:
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@@
 <drawing>
 <settings>
-<setting alwaysvectorfont="no"/>
+<setting alwaysvectorfont="yes"/>
 <setting verticaltext="up"/>
 </settings>
@@
 <wire x1="23.752040625" y1="24.0583" x2="23.9798" y2="23.2083" width="0.001" layer="20"/>
 <text x="87.884" y="3.81" size="1.524" layer="25" font="vector" ratio="15">word</text>
+<text x="35.814" y="82.677" size="2.032" layer="22" font="vector" ratio="20" rot="SMR0">GND</text>
+<text x="30.734" y="82.677" size="2.032" layer="21" font="vector" ratio="20" rot="SR0">GND</text>
+<text x="28.702" y="53.594" size="1.524" layer="21" font="vector" ratio="20" rot="SR270">hippo-pd monitor v1</text>
+<text x="28.702" y="86.233" size="1.524" layer="21" font="vector" ratio="20" rot="SR270">ek robotgrrl Jul 22, '22</text>
+<text x="28.702" y="53.594" size="1.524" layer="22" font="vector" ratio="20" rot="SR270">hippo-pd monitor v1</text>
+<text x="28.448" y="86.233" size="1.524" layer="22" font="vector" ratio="20" rot="SR270">ek robotgrrl Jul 22, '22</text>
+<text x="114.554" y="32.131" size="2.032" layer="22" font="vector" ratio="20" rot="SMR0">GND</text>
+<text x="109.474" y="32.131" size="2.032" layer="21" font="vector" ratio="20" rot="SR0">GND</text>
+<text x="36.576" y="32.385" size="2.032" layer="22" font="vector" ratio="20" rot="SMR0">IN+</text>
+<text x="31.496" y="32.385" size="2.032" layer="21" font="vector" ratio="20" rot="SR0">IN+</text>
+<text x="115.062" y="81.661" size="2.032" layer="22" font="vector" ratio="20" rot="SMR0">IN+</text>
+<text x="109.982" y="81.661" size="2.032" layer="21" font="vector" ratio="20" rot="SR0">IN+</text>
 </plain>
 <attributes>
@@
 </element>
 <element name="TP1" library="Hippo-PS" package="TP" value="TP" x="33.528" y="36.068" smashed="yes">
-<attribute name="NAME" x="36.576" y="36.83" size="1.778" layer="25" font="vector" ratio="14"/>
-<attribute name="VALUE" x="37.338" y="33.528" size="1.778" layer="25" font="vector" ratio="14"/>
+<attribute name="NAME" x="36.068" y="36.576" size="1.778" layer="25" font="vector" ratio="14"/>
+<attribute name="VALUE" x="19.304" y="39.878" size="1.778" layer="25" font="vector" ratio="14"/>
 </element>
 <element name="TP2" library="Hippo-PS" package="TP" value="TP" x="33.528" y="80.518" smashed="yes">
-<attribute name="NAME" x="37.338" y="81.788" size="1.778" layer="25" font="vector" ratio="14"/>
-<attribute name="VALUE" x="37.338" y="77.978" size="1.778" layer="25" font="vector" ratio="14"/>
+<attribute name="NAME" x="36.322" y="78.232" size="1.778" layer="25" font="vector" ratio="14"/>
+<attribute name="VALUE" x="17.526" y="75.438" size="1.778" layer="25" font="vector" ratio="14"/>
 </element>
 <element name="Q1" library="Hippo-PS" package="PN2222A-SOT-23" value="PN2222A-SOT-23" x="113.03" y="61.722" smashed="yes" rot="R90">
@@
 </element>
 <element name="TP6" library="Hippo-PS" package="TP" value="TP" x="79.248" y="24.13" smashed="yes">
-<attribute name="NAME" x="83.058" y="25.4" size="1.778" layer="25" font="vector" ratio="14"/>
-<attribute name="VALUE" x="83.058" y="21.59" size="1.778" layer="25" font="vector" ratio="14"/>
+<attribute name="NAME" x="77.216" y="19.304" size="1.778" layer="25" font="vector" ratio="14"/>
+<attribute name="VALUE" x="80.01" y="14.224" size="1.778" layer="25" font="vector" ratio="14"/>
 </element>
 <element name="S2" library="Hippo-PS" package="TACTILE_BUTTON" value="TACTILE_BUTTON" x="76.454" y="53.34" smashed="yes" rot="R90">
@@
 <wire x1="48.768" y1="67.818" x2="48.768" y2="65.024" width="0.3048" layer="1"/>
 <wire x1="84.328" y1="80.264" x2="84.328" y2="77.47" width="0.3048" layer="1"/>
-<wire x1="85.09" y1="94.036" x2="99.314" y2="94.036" width="0" layer="19" extent="1-1"/>
-<wire x1="84.328" y1="80.264" x2="85.09" y2="94.036" width="0" layer="19" extent="1-1"/>
-<wire x1="70.866" y1="94.036" x2="85.09" y2="94.036" width="0" layer="19" extent="1-1"/>
-<wire x1="56.134" y1="94.036" x2="70.866" y2="94.036" width="0" layer="19" extent="1-1"/>
-<wire x1="70.01" y1="72.644" x2="84.328" y2="77.47" width="0" layer="19" extent="1-1"/>
-<wire x1="54.864" y1="58.166" x2="70.01" y2="72.644" width="0" layer="19" extent="1-1"/>
-<wire x1="48.768" y1="65.024" x2="54.864" y2="58.166" width="0" layer="19" extent="1-1"/>
-<wire x1="42.164" y1="43.362" x2="54.864" y2="58.166" width="0" layer="19" extent="1-1"/>
-<wire x1="39.116" y1="43.362" x2="42.164" y2="43.362" width="0" layer="19" extent="1-1"/>
-<wire x1="33.528" y1="80.518" x2="48.768" y2="67.818" width="0" layer="19" extent="1-1"/>
-<wire x1="32.258" y1="93.218" x2="33.528" y2="80.518" width="0" layer="19" extent="1-1"/>
-<wire x1="45.212" y1="20.598" x2="42.164" y2="43.362" width="0" layer="19" extent="1-1"/>
-<wire x1="48.26" y1="20.598" x2="45.212" y2="20.598" width="0" layer="19" extent="1-1"/>
-<wire x1="51.308" y1="20.598" x2="48.26" y2="20.598" width="0" layer="19" extent="1-1"/>
-<wire x1="54.356" y1="20.598" x2="51.308" y2="20.598" width="0" layer="19" extent="1-1"/>
-<wire x1="57.404" y1="20.598" x2="54.356" y2="20.598" width="0" layer="19" extent="1-1"/>
-<wire x1="60.452" y1="20.598" x2="57.404" y2="20.598" width="0" layer="19" extent="1-1"/>
-<wire x1="63.5" y1="20.598" x2="60.452" y2="20.598" width="0" layer="19" extent="1-1"/>
-<wire x1="66.548" y1="20.598" x2="63.5" y2="20.598" width="0" layer="19" extent="1-1"/>
-<wire x1="69.596" y1="20.598" x2="66.548" y2="20.598" width="0" layer="19" extent="1-1"/>
-<wire x1="72.644" y1="20.598" x2="69.596" y2="20.598" width="0" layer="19" extent="1-1"/>
-<wire x1="79.248" y1="24.13" x2="72.644" y2="20.598" width="0" layer="19" extent="1-1"/>
-<wire x1="80.264" y1="34.29" x2="79.248" y2="24.13" width="0" layer="19" extent="1-1"/>
-<wire x1="74.93" y1="43.362" x2="78.232" y2="43.362" width="0" layer="19" extent="1-1"/>
-<wire x1="89.766" y1="21.096" x2="79.248" y2="24.13" width="0" layer="19" extent="1-1"/>
-<wire x1="91.186" y1="45.648" x2="80.01" y2="41.148" width="0" layer="19" extent="1-1"/>
-<wire x1="94.488" y1="45.648" x2="91.186" y2="45.648" width="0" layer="19" extent="1-1"/>
-<wire x1="97.536" y1="34.234" x2="94.488" y2="45.648" width="0" layer="19" extent="1-1"/>
-<wire x1="110.316" y1="47.244" x2="94.488" y2="45.648" width="0" layer="19" extent="1-1"/>
-<wire x1="114.01" y1="62.672" x2="110.316" y2="47.244" width="0" layer="19" extent="1-1"/>
-<wire x1="112.268" y1="23.241" x2="97.536" y2="34.234" width="0" layer="19" extent="1-1"/>
 </signal>
 <signal name="N$6">

Commit message: Updated refdes of some components
Parts:
- D1, D10, D9: value GREEN -> BLUE
- D6: value BLUE -> GREEN
- renumbered U$1 to U1, U$2 to U2
